Commit message: Created core URDF

File: description/lidar.xacro (robot description, xacro)
@@ -23,4 +23,5 @@
     </link>
     <gazebo reference="laser_frame">
+        <material>Gazebo/Red</material>
         <sensor name="laser" type="ray">
             <pose> 0 0 0 0 0 0 </pose>
@@ -32,5 +33,5 @@
                         <samples>360</samples>
                         <resolution>1</resolution>
-                        <min_angle>3.14</min_angle>
+                        <min_angle>-3.14</min_angle>
                         <max_angle>3.14</max_angle>
                     </horizontal>
