Commit message: Created core URDF

File: description/robot.urdf.xacro (robot description, xacro)
@@ -1,9 +1,14 @@
 <?xml version="1.0"?>
 <robot xmlns:xacro="http://www.ros.org/wiki/xacro"  name="robot">
+    <xacro:arg name="use_ros2_control" default="true"/>
     <xacro:include filename="robot_core.xacro" />
-    <!-- <xacro:include filename="gazebo_control.xacro" /> -->
+    <xacro:if value="$(arg use_ros2_control)">
+        <xacro:include filename="ros2_control.xacro" />
+    </xacro:if>
+    <xacro:unless value="$(arg use_ros2_control)">
+        <xacro:include filename="gazebo_control.xacro" />
+    </xacro:unless>
     <xacro:include filename="lidar.xacro" />
-    <!-- <xacro:include filename="camera.xacro" /> -->
-    <xacro:include filename="depth_camera.xacro" />
-    <xacro:include filename="ros2_control.xacro" />
+    <xacro:include filename="camera.xacro" />
+    <!-- <xacro:include filename="depth_camera.xacro" /> -->
 </robot>

File: description/robot_core.xacro (robot description, xacro)
@@ -16,12 +16,12 @@
     <xacro:property name="caster_wheel_offset_x" value="0.075"/>
     <xacro:property name="caster_wheel_offset_z" value="${wheel_offset_z - wheel_radius + caster_wheel_radius}"/>
-    <material name="transparent">
-        <color rgba="1 1 1 0.5" />
-    </material>
-    <material name="yellow">
-        <color rgba="1 1 0 1"/>
+    <material name="white">
+        <color rgba="1 1 1 1" />
     </material>
     <material name="blue">
         <color rgba="0.2 0.2 1 1"/>
+    </material>
+    <material name="orange">
+        <color rgba="1 0.3 0.1 1"/>
     </material>
     <material name="black">
@@ -46,5 +46,5 @@
                 <box size="${chassis_length} ${chassis_width} ${chassis_height}"/>
             </geometry>
-            <material name="transparent"/>
+            <material name="orange"/>
         </visual>
         <collision>
@@ -59,5 +59,5 @@
     </link>
     <gazebo reference="chassis">
-        <material>Gazebo/Transparent</material>
+        <material>Gazebo/Orange</material>
     </gazebo>
     <!-- LEFT WHEEL LINK -->
@@ -73,5 +73,5 @@
                 <cylinder radius="${wheel_radius}" length="${wheel_thickness}"/>
             </geometry>
-            <material name="yellow"/>
+            <material name="blue"/>
         </visual>
         <collision>
@@ -85,5 +85,5 @@
     </link>
     <gazebo reference="left_wheel">
-        <material>Gazebo/Yellow</material>
+        <material>Gazebo/Blue</material>
     </gazebo>
     <!-- RIGHT WHEEL LINK -->
@@ -99,5 +99,5 @@
                 <cylinder radius="${wheel_radius}" length="${wheel_thickness}"/>
             </geometry>
-            <material name="yellow"/>
+            <material name="blue"/>
         </visual>
         <collision>
@@ -111,5 +111,5 @@
     </link>
     <gazebo reference="right_wheel">
-        <material>Gazebo/Yellow</material>
+        <material>Gazebo/Blue</material>
     </gazebo>
     <!-- CASTER WHEEL LINK -->
